File: flatbox.kicad_sch (KiCad schematic)
At the start: 31 parts, among them J3 USB_C_Receptacle_USB2.0_16P, SW1 SW_Push, SW10 SW_Push, SW2 SW_Push, SW3 SW_Push, SW4 SW_Push, SW5 SW_Push, SW6 SW_Push, SW7 SW_Push, SW8 SW_Push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

Commit message: Second Commit done, some updates to the schematic have been made
Parts:
- removed C4, C5: 22pF, symbol Device:C_Polarized_US
- removed Y2: Crystal_GND23, symbol Device:Crystal_GND23
- added C2, C3: 22pF, symbol Device:C
- added Y1: 16MHz, symbol Device:Crystal
- R10, R11, R12, R13, R16, R5, R6, R7, R8, R9: value 1k -> 10k
Connections:
- net +5V: now also R10.2, R11.2, R12.2, R13.2, R16.2, R5.2, R6.2, R7.2, R8.2, R9.2
- net 1+2: now also SW9.2
- net 3+4: now also SW10.2
- net CIRCLE: now also SW4.2
- net CROSS: now also SW3.2
- net DOWN: now also SW6.2
- net GND: now also SW1.1, SW10.1, SW2.1, SW3.1, SW4.1, SW5.1, SW6.1, SW7.1, SW8.1, SW9.1, C2.1, C3.1; no longer SW1.2, SW10.2, SW2.2, SW3.2, SW4.2, SW5.2, SW6.2, SW7.2, SW8.2, SW9.2
- net LEFT: now also SW7.2
- net RIGHT: now also SW8.2
- net SQUARE: now also SW1.2
- net TRIANGLE: now also SW2.2
- net UP: now also SW5.2
- net at U1.16 (XTAL2): now also C3.2, Y1.1
- net at U1.17 (XTAL1): now also C2.2, Y1.2
Other:
- moved on the sheet: R10, R11, R12, R13, R16, R5, R6, R7, R8, R9, SW1, SW10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
