File: flatbox.kicad_sch (KiCad schematic)
At the start: 31 parts, among them J3 USB_C_Receptacle_USB2.0_16P, SW1 SW_Push, SW10 SW_Push, SW2 SW_Push, SW3 SW_Push, SW4 SW_Push, SW5 SW_Push, SW6 SW_Push, SW7 SW_Push, SW8 SW_Push, SW9 SW_Push, U1 ATmega32U4-A, Y1 16MHz

Commit message: Modified schematic
Parts:
- added R17: 10k, symbol Device:R
Connections:
- net +5V: now also R17.2
- net at U1.13 (~{RESET}): now also R17.1
- no-connect marks 2 -> 4
