File: flatbox.kicad_sch (KiCad schematic)
At the start: 35 parts, among them J3 USB_C_Receptacle_USB2.0_16P, SW1 SW_Push, SW10 SW_Push, SW11 SW_Push, SW2 SW_Push, SW3 SW_Push, SW4 SW_Push, SW5 SW_Push, SW6 SW_Push, SW7 SW_Push, SW8 SW_Push, SW9 SW_Push, U1 ATmega32U4-A, Y1 16MHz

Commit message: Added PCB Components of Schematic
Parts:
- J3: footprint Connector_USB:USB_C_Receptacle_HRO_TYPE-C-31-M-12 -> Library:USB_C_Receptacle_HRO_TYPE-C-31-M-12
- SW1, SW10, SW11, SW2, SW3, SW4, SW5, SW6, SW7, SW8, SW9: footprint (none) -> Button_Switch_Keyboard:SW_Cherry_MX_1.00u_PCB
- Y1: footprint (none) -> Crystal:Crystal_HC49-4H_Vertical
Changed lines of the file:
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@@
 			)
 		)
-		(property "Footprint" ""
+		(property "Footprint" "Button_Switch_Keyboard:SW_Cherry_MX_1.00u_PCB"
 			(at 41.91 156.21 0)
 			(hide yes)
@@
 			)
 		)
-		(property "Footprint" ""
+		(property "Footprint" "Button_Switch_Keyboard:SW_Cherry_MX_1.00u_PCB"
 			(at 41.91 168.91 0)
 			(hide yes)
@@
 			)
 		)
-		(property "Footprint" ""
+		(property "Footprint" "Button_Switch_Keyboard:SW_Cherry_MX_1.00u_PCB"
 			(at 41.91 83.82 0)
 			(hide yes)
@@
 			)
 		)
-		(property "Footprint" ""
+		(property "Footprint" "Button_Switch_Keyboard:SW_Cherry_MX_1.00u_PCB"
 			(at 41.91 105.41 0)
 			(hide yes)
@@
 			)
 		)
-		(property "Footprint" ""
+		(property "Footprint" "Button_Switch_Keyboard:SW_Cherry_MX_1.00u_PCB"
 			(at 41.91 179.07 0)
 			(hide yes)
@@
 			)
 		)
-		(property "Footprint" ""
+		(property "Footprint" "Button_Switch_Keyboard:SW_Cherry_MX_1.00u_PCB"
 			(at 41.91 93.98 0)
 			(hide yes)
@@
 			)
 		)
-		(property "Footprint" ""
+		(property "Footprint" "Button_Switch_Keyboard:SW_Cherry_MX_1.00u_PCB"
 			(at 41.91 143.51 0)
 			(hide yes)
@@
 			)
 		)
-		(property "Footprint" "Connector_USB:USB_C_Receptacle_HRO_TYPE-C-31-M-12"
+		(property "Footprint" "Library:USB_C_Receptacle_HRO_TYPE-C-31-M-12"
 			(at 33.02 43.18 0)
 			(hide yes)
@@
 			)
 		)
-		(property "Footprint" ""
+		(property "Footprint" "Button_Switch_Keyboard:SW_Cherry_MX_1.00u_PCB"
 			(at 41.91 132.08 0)
 			(hide yes)
@@
 			)
 		)
-		(property "Footprint" ""
+		(property "Footprint" "Button_Switch_Keyboard:SW_Cherry_MX_1.00u_PCB"
 			(at 199.39 39.37 0)
 			(hide yes)
@@
 			)
 		)
-		(property "Footprint" ""
+		(property "Footprint" "Button_Switch_Keyboard:SW_Cherry_MX_1.00u_PCB"
 			(at 41.91 187.96 0)
 			(hide yes)
@@
 			)
 		)
-		(property "Footprint" ""
+		(property "Footprint" "Crystal:Crystal_HC49-4H_Vertical"
 			(at 209.55 58.42 0)
 			(hide yes)
@@
 			)
 		)
-		(property "Footprint" ""
+		(property "Footprint" "Button_Switch_Keyboard:SW_Cherry_MX_1.00u_PCB"
 			(at 41.91 118.11 0)
 			(hide yes)

Commit message: Updated Schematic and PCB
Parts:
- added R18, R19: 10k, Resistor_SMD:R_0805_2012Metric, symbol Device:R
- added SW12, SW13: SW_Push, Button_Switch_Keyboard:SW_Cherry_MX_1.00u_PCB, symbol Switch:SW_Push
Connections:
- net +5V: now also R18.2, R19.2
- net GND: now also SW12.1, SW13.1
- net 2+4: now reaches U1.31 (PC6)
- net 2+4: now also R18.1, SW12.2
- net 1+3: now reaches U1.32 (PC7)
- net 1+3: now also R19.1, SW13.2
- no-connect marks 19 -> 17

Commit message: Updated PCB & Schematic
Connections:
- net +5V: now also R13.1; no longer R13.2
- net 1+2: now also R13.2; no longer R13.1
Other:
- moved on the sheet: R13
Changed lines of the file:
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@@
 	(symbol
 		(lib_id "Device:R")
-		(at 55.88 184.15 90)
+		(at 55.88 184.15 270)
+		(mirror x)
 		(unit 1)
 		(body_style 1)
@@
 		)
 		(property "Value" "10k"
-			(at 56.134 184.15 90)
+			(at 55.626 184.15 90)
 			(show_name no)
 			(do_not_autoplace no)

Commit message: Modified Schematic and PCB Assembly
Parts:
- added J1: Conn_01x06_Pin, symbol Connector:Conn_01x06_Pin
- added R20: 10k, Resistor_SMD:R_0805_2012Metric, symbol Device:R
- added SW14: SW_Push, Button_Switch_Keyboard:SW_Cherry_MX_1.00u_PCB, symbol Switch:SW_Push
Connections:
- net +5V: now also J1.1 (Pin_1), R20.2
- net GND: now also J1.6 (Pin_6), SW14.1
- net RESET: now reaches R17.1, SW11.2, U1.13 (~{RESET})
- net RESET: now also J1.5 (Pin_5)
- net START: now reaches U1.20 (PD2)
- net START: now also R20.1, SW14.2
- net CIRCLE renamed CIRCLE/MISO
- net CIRCLE/MISO: now also J1.4 (Pin_4)
- net CROSS renamed CROSS/MOSI
- net CROSS/MOSI: now also J1.3 (Pin_3)
- net TRIANGLE renamed TRIANGLE/SCK
- net TRIANGLE/SCK: now also J1.2 (Pin_2)
- no-connect marks 17 -> 16
Other:
- note added: "Connections"
