File: flatbox.kicad_pcb (KiCad board)
At the start: 2 copper layers, 35 parts, among them J3 USB_C_Receptacle_USB2.0_16P, SW1 SW_Push, SW10 SW_Push, SW11 SW_Push, SW2 SW_Push, SW3 SW_Push, SW4 SW_Push, SW5 SW_Push, SW6 SW_Push, SW7 SW_Push, SW8 SW_Push, SW9 SW_Push, U1 ATmega32U4-A, Y1 16MHz

Commit message: Updated Schematic and PCB
Parts:
- added R18: 10k, Resistor_SMD:R_0805_2012Metric, F.Cu at (279.6, 139.5)
- added R19: 10k, Resistor_SMD:R_0805_2012Metric, F.Cu at (279.6, 142.4)
- added SW12: SW_Push, Button_Switch_Keyboard:SW_Cherry_MX_1.00u_PCB, F.Cu at (316.6, 70.9)
- added SW13: SW_Push, Button_Switch_Keyboard:SW_Cherry_MX_1.00u_PCB, F.Cu at (308.6, 108.9)
- moved SW9 182.0 mm to (273.6, 108.4)
- moved SW10 179.0 mm to (281.0, 70.9)
- moved SW2 174.6 mm to (246.3, 72.5)
- moved SW4 168.3 mm to (239.5, 109.4)
- moved SW5 156.6 mm to (193.0, 162.4)
- moved SW1 148.0 mm to (215.0, 85.4)
- moved SW3 142.8 mm to (208.0, 120.9)
- moved R15 110.2 mm to (228.5, 62.7)
- moved R16 110.2 mm to (228.5, 65.6)
- moved R3 110.2 mm to (219.7, 62.7)
- moved R4 110.2 mm to (219.7, 65.6)
- moved R5 110.2 mm to (219.7, 68.6)
- moved R6 110.2 mm to (219.7, 71.5)
- moved R7 110.2 mm to (219.7, 74.5)
- moved R8 110.2 mm to (219.7, 77.4)
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Connections:
- U1 pad 31: unconnected-(U1-PC6-Pad31) -> /2+4
- U1 pad 32: unconnected-(U1-PC7-Pad32) -> /1+3
Other:
- board outline added: 296 x 196 mm
