File: flatbox.kicad_pcb (KiCad board)
At the start: 2 copper layers, 296 x 196 mm, 39 parts, among them J3 USB_C_Receptacle_USB2.0_16P, SW1 SW_Push, SW10 SW_Push, SW11 SW_Push, SW12 SW_Push, SW13 SW_Push, SW2 SW_Push, SW3 SW_Push, SW4 SW_Push, SW5 SW_Push, SW6 SW_Push, SW7 SW_Push, SW8 SW_Push, SW9 SW_Push, U1 ATmega32U4-A, Y1 16MHz

Commit message: Updated PCB & Schematic
Parts:
- moved R9 100.8 mm to (184.0, 156.5), turned to 0 degrees
- moved R17 84.8 mm to (97.0, 63.0)
- moved R13 82.8 mm to (260.5, 107.5), turned to 90 degrees
- moved R6 4.00 mm to (233.0, 72.0)
- moved C3 3.69 mm to (181.5, 64.5)
- moved C5 1.22 mm to (178.5, 61.5), turned to 90 degrees
- moved C4 0.87 mm to (178.5, 57.5), turned to 90 degrees
- moved C1 0.64 mm to (178.5, 53.5), turned to -90 degrees
Routing:
- net +5V: track 14.6 -> 358.0 mm
- net GND: track 74.5 -> 0.06 mm
- net Net-(U1-~{RESET}): track 0.00 -> 14.0 mm
- net /SQUARE: track 0.00 -> 10.6 mm
- net /UP: track 0.00 -> 9.95 mm
- net Net-(J3-CC1): track 0.00 -> 9.76 mm
- net /1+3: track 0.00 -> 8.33 mm
- net /2+4: track 0.00 -> 8.08 mm
- net /CIRCLE: track 0.00 -> 8.00 mm
- net Net-(J3-CC2): track 0.00 -> 7.92 mm
- net /TRIANGLE: track 0.00 -> 7.86 mm
- net /CROSS: track 0.00 -> 7.83 mm
- net /1+2: track 0.00 -> 7.83 mm
- net /3+4: track 0.00 -> 7.41 mm
- net Net-(U1-XTAL1): track 0.00 -> 6.82 mm
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